Commit message: changed joint limits and updated model

File: resources/models/iCubGenova04.urdf (robot description, URDF)
Before this commit: robot iCub, 163 links, 162 joints
Links:
- removed link chest_ems_acc_eb1
- removed link chest_ems_acc_eb2
- removed link chest_ems_acc_eb3
- removed link chest_ems_acc_eb4
- removed link chest_ems_gyro_eb1
- removed link chest_ems_gyro_eb2
- removed link chest_ems_gyro_eb3
- removed link chest_ems_gyro_eb4
- removed link chest_mtb_acc_0b10
- removed link chest_mtb_acc_0b7
- removed link chest_mtb_acc_0b8
- removed link chest_mtb_acc_0b9
- removed link l_foot_mtb_acc_10b12
- removed link l_foot_mtb_acc_10b13
- removed link l_forearm_mtb_acc_1b7
- removed link l_forearm_mtb_acc_1b8
- removed link l_forearm_mtb_acc_1b9
- removed link l_lower_leg_ems_acc_eb7
- removed link l_lower_leg_ems_gyro_eb7
- removed link l_lower_leg_mtb_acc_10b10
- removed link l_lower_leg_mtb_acc_10b11
- removed link l_lower_leg_mtb_acc_10b8
- removed link l_lower_leg_mtb_acc_10b9
- removed link l_upper_arm_mtb_acc_1b10
- removed link l_upper_arm_mtb_acc_1b11
- removed link l_upper_arm_mtb_acc_1b12
- removed link l_upper_arm_mtb_acc_1b13
- removed link l_upper_leg_ems_acc_eb10
- removed link l_upper_leg_ems_acc_eb6
- removed link l_upper_leg_ems_gyro_eb10
- removed link l_upper_leg_ems_gyro_eb6
- removed link l_upper_leg_mtb_acc_10b1
- removed link l_upper_leg_mtb_acc_10b2
- removed link l_upper_leg_mtb_acc_10b3
- removed link l_upper_leg_mtb_acc_10b4
- removed link l_upper_leg_mtb_acc_10b5
- removed link l_upper_leg_mtb_acc_10b6
- removed link l_upper_leg_mtb_acc_10b7
- removed link r_foot_mtb_acc_11b12
- removed link r_foot_mtb_acc_11b13
- removed link r_forearm_mtb_acc_2b7
- removed link r_forearm_mtb_acc_2b8
- removed link r_forearm_mtb_acc_2b9
- removed link r_lower_leg_ems_acc_eb9
- removed link r_lower_leg_ems_gyro_eb9
- removed link r_lower_leg_mtb_acc_11b10
- removed link r_lower_leg_mtb_acc_11b11
- removed link r_lower_leg_mtb_acc_11b8
- removed link r_lower_leg_mtb_acc_11b9
- removed link r_upper_arm_mtb_acc_2b10
- removed link r_upper_arm_mtb_acc_2b11
- removed link r_upper_arm_mtb_acc_2b12
- removed link r_upper_arm_mtb_acc_2b13
- removed link r_upper_leg_ems_acc_eb11
- removed link r_upper_leg_ems_acc_eb8
- removed link r_upper_leg_ems_gyro_eb11
- removed link r_upper_leg_ems_gyro_eb8
- removed link r_upper_leg_mtb_acc_11b1
- removed link r_upper_leg_mtb_acc_11b2
- removed link r_upper_leg_mtb_acc_11b3
- removed link r_upper_leg_mtb_acc_11b4
- removed link r_upper_leg_mtb_acc_11b5
- removed link r_upper_leg_mtb_acc_11b6
- removed link r_upper_leg_mtb_acc_11b7
- removed link root_link_ems_acc_eb5
- removed link root_link_ems_gyro_eb5
Joints:
- removed joint chest_ems_acc_eb1_fixed_joint
- removed joint chest_ems_acc_eb2_fixed_joint
- removed joint chest_ems_acc_eb3_fixed_joint
- removed joint chest_ems_acc_eb4_fixed_joint
- removed joint chest_ems_gyro_eb1_fixed_joint
- removed joint chest_ems_gyro_eb2_fixed_joint
- removed joint chest_ems_gyro_eb3_fixed_joint
- removed joint chest_ems_gyro_eb4_fixed_joint
- removed joint chest_mtb_acc_0b10_fixed_joint
- removed joint chest_mtb_acc_0b7_fixed_joint
- removed joint chest_mtb_acc_0b8_fixed_joint
- removed joint chest_mtb_acc_0b9_fixed_joint
- removed joint l_foot_mtb_acc_10b12_fixed_joint
- removed joint l_foot_mtb_acc_10b13_fixed_joint
- removed joint l_forearm_mtb_acc_1b7_fixed_joint
- removed joint l_forearm_mtb_acc_1b8_fixed_joint
- removed joint l_forearm_mtb_acc_1b9_fixed_joint
- removed joint l_lower_leg_ems_acc_eb7_fixed_joint
- removed joint l_lower_leg_ems_gyro_eb7_fixed_joint
- removed joint l_lower_leg_mtb_acc_10b10_fixed_joint
- removed joint l_lower_leg_mtb_acc_10b11_fixed_joint
- removed joint l_lower_leg_mtb_acc_10b8_fixed_joint
- removed joint l_lower_leg_mtb_acc_10b9_fixed_joint
- removed joint l_upper_arm_mtb_acc_1b10_fixed_joint
- removed joint l_upper_arm_mtb_acc_1b11_fixed_joint
- removed joint l_upper_arm_mtb_acc_1b12_fixed_joint
- removed joint l_upper_arm_mtb_acc_1b13_fixed_joint
- removed joint l_upper_leg_ems_acc_eb10_fixed_joint
- removed joint l_upper_leg_ems_acc_eb6_fixed_joint
- removed joint l_upper_leg_ems_gyro_eb10_fixed_joint
- removed joint l_upper_leg_ems_gyro_eb6_fixed_joint
- removed joint l_upper_leg_mtb_acc_10b1_fixed_joint
- removed joint l_upper_leg_mtb_acc_10b2_fixed_joint
- removed joint l_upper_leg_mtb_acc_10b3_fixed_joint
- removed joint l_upper_leg_mtb_acc_10b4_fixed_joint
- removed joint l_upper_leg_mtb_acc_10b5_fixed_joint
- removed joint l_upper_leg_mtb_acc_10b6_fixed_joint
- removed joint l_upper_leg_mtb_acc_10b7_fixed_joint
- removed joint r_foot_mtb_acc_11b12_fixed_joint
- removed joint r_foot_mtb_acc_11b13_fixed_joint
- removed joint r_forearm_mtb_acc_2b7_fixed_joint
- removed joint r_forearm_mtb_acc_2b8_fixed_joint
- removed joint r_forearm_mtb_acc_2b9_fixed_joint
- removed joint r_lower_leg_ems_acc_eb9_fixed_joint
- removed joint r_lower_leg_ems_gyro_eb9_fixed_joint
- removed joint r_lower_leg_mtb_acc_11b10_fixed_joint
- removed joint r_lower_leg_mtb_acc_11b11_fixed_joint
- removed joint r_lower_leg_mtb_acc_11b8_fixed_joint
- removed joint r_lower_leg_mtb_acc_11b9_fixed_joint
- removed joint r_upper_arm_mtb_acc_2b10_fixed_joint
- removed joint r_upper_arm_mtb_acc_2b11_fixed_joint
- removed joint r_upper_arm_mtb_acc_2b12_fixed_joint
- removed joint r_upper_arm_mtb_acc_2b13_fixed_joint
- removed joint r_upper_leg_ems_acc_eb11_fixed_joint
- removed joint r_upper_leg_ems_acc_eb8_fixed_joint
- removed joint r_upper_leg_ems_gyro_eb11_fixed_joint
- removed joint r_upper_leg_ems_gyro_eb8_fixed_joint
- removed joint r_upper_leg_mtb_acc_11b1_fixed_joint
- removed joint r_upper_leg_mtb_acc_11b2_fixed_joint
- removed joint r_upper_leg_mtb_acc_11b3_fixed_joint
- removed joint r_upper_leg_mtb_acc_11b4_fixed_joint
- removed joint r_upper_leg_mtb_acc_11b5_fixed_joint
- removed joint r_upper_leg_mtb_acc_11b6_fixed_joint
- removed joint r_upper_leg_mtb_acc_11b7_fixed_joint
- removed joint root_link_ems_acc_eb5_fixed_joint
- removed joint root_link_ems_gyro_eb5_fixed_joint
- joint l_ankle_pitch: limit lower=-0.349065850399 upper=0.523598775598 effort=50000 velocity=50000 -> lower=-0.523598775598 upper=0.523598775598 effort=50000 velocity=50000
- joint l_hip_roll: limit lower=0.0 upper=1.57079632679 effort=50000 velocity=50000 -> lower=-0.261799 upper=1.48353 effort=50000 velocity=50000
- joint r_ankle_pitch: limit lower=-0.349065850399 upper=0.523598775598 effort=50000 velocity=50000 -> lower=-0.523598775598 upper=0.523598775598 effort=50000 velocity=50000
- joint r_hip_roll: limit lower=0.0 upper=1.57079632679 effort=50000 velocity=50000 -> lower=-0.261799 upper=1.48353 effort=50000 velocity=50000

Commit message: update model to the newest version

File: resources/models/iCubGenova04.urdf (robot description, URDF)
Before this commit: robot iCub, 97 links, 96 joints
Links:
- added link l_upper_leg_back_contact
- added link l_upper_leg_dh_frame
- added link r_lower_leg_skin_0
- added link r_lower_leg_skin_10
- added link r_lower_leg_skin_11
- added link r_lower_leg_skin_14
- added link r_lower_leg_skin_15
- added link r_lower_leg_skin_16
- added link r_lower_leg_skin_17
- added link r_lower_leg_skin_19
- added link r_lower_leg_skin_20
- added link r_lower_leg_skin_21
- added link r_lower_leg_skin_28
- added link r_lower_leg_skin_29
- added link r_lower_leg_skin_3
- added link r_lower_leg_skin_31
- added link r_lower_leg_skin_32
- added link r_lower_leg_skin_35
- added link r_lower_leg_skin_36
- added link r_lower_leg_skin_37
- added link r_lower_leg_skin_38
- added link r_lower_leg_skin_4
- added link r_lower_leg_skin_41
- added link r_lower_leg_skin_42
- added link r_lower_leg_skin_43
- added link r_lower_leg_skin_46
- added link r_lower_leg_skin_47
- added link r_lower_leg_skin_49
- added link r_lower_leg_skin_5
- added link r_lower_leg_skin_50
- added link r_lower_leg_skin_51
- added link r_lower_leg_skin_52
- added link r_lower_leg_skin_53
- added link r_lower_leg_skin_54
- added link r_lower_leg_skin_55
- added link r_lower_leg_skin_56
- added link r_lower_leg_skin_6
- added link r_lower_leg_skin_60
- added link r_lower_leg_skin_61
- added link r_lower_leg_skin_9
- added link r_upper_leg_back_contact
- added link r_upper_leg_dh_frame
- link l_foot: mass 0.382372 -> 0.382968
- link l_hip_1: mass 0.915608 -> 0.919725
- link l_hip_2: mass 0.421161 -> 0.421106
- link r_foot: mass 0.38227 -> 0.382866
- link r_hip_1: mass 0.920101 -> 0.919978
- link r_hip_2: mass 0.4194 -> 0.418361
Joints:
- added joint l_upper_leg_back_contact_fixed_joint: type fixed, parent l_upper_leg, child l_upper_leg_back_contact, origin xyz=-0.0512567 0 0.0146 rpy=0 1.57079632679 0
- added joint l_upper_leg_dh_frame_fixed_joint: type fixed, parent l_upper_leg, child l_upper_leg_dh_frame, origin xyz=0 0 -0.145825 rpy=1.57079632679 0 0
- added joint r_lower_leg_skin_0_fixed_joint: type fixed, parent r_lower_leg, child r_lower_leg_skin_0, origin xyz=0.0544117 -0.031214 -0.002634 rpy=2.09173809157e-06 -1.41530676247 2.48648458622
- added joint r_lower_leg_skin_10_fixed_joint: type fixed, parent r_lower_leg, child r_lower_leg_skin_10, origin xyz=0.0644607 0.0003424 -0.021205 rpy=3.14159265355 -1.47095803541 0.000430021675261
- added joint r_lower_leg_skin_11_fixed_joint: type fixed, parent r_lower_leg, child r_lower_leg_skin_11, origin xyz=0.0607108 -0.0160916 -0.030885 rpy=-3.14159218252 -1.3281180406 -0.27213836788
- added joint r_lower_leg_skin_14_fixed_joint: type fixed, parent r_lower_leg, child r_lower_leg_skin_14, origin xyz=0.0550477 -0.031176 -0.0219 rpy=-3.14159181885 -1.46502735635 -0.654033407167
- added joint r_lower_leg_skin_15_fixed_joint: type fixed, parent r_lower_leg, child r_lower_leg_skin_15, origin xyz=0.0591708 -0.0161788 0.007243 rpy=4.27484256729e-07 -1.25203633076 2.86798859471
- added joint r_lower_leg_skin_16_fixed_joint: type fixed, parent r_lower_leg, child r_lower_leg_skin_16, origin xyz=0.0272875 -0.050287 -0.004549 rpy=1.33075915123e-05 -1.53260853515 1.96280242835
- added joint r_lower_leg_skin_17_fixed_joint: type fixed, parent r_lower_leg, child r_lower_leg_skin_17, origin xyz=0.027875 -0.050312 -0.023882 rpy=-3.1415645262 -1.56366240237 -1.18022508756
- added joint r_lower_leg_skin_19_fixed_joint: type fixed, parent r_lower_leg, child r_lower_leg_skin_19, origin xyz=0.0357534 0.0410628 0.006065 rpy=-8.90877717426e-07 -1.43498696978 -2.15863618017
- added joint r_lower_leg_skin_20_fixed_joint: type fixed, parent r_lower_leg, child r_lower_leg_skin_20, origin xyz=0.0234419 0.0479908 -0.004952 rpy=-3.20556549428e-06 -1.50015513031 -1.86755092413
- added joint r_lower_leg_skin_21_fixed_joint: type fixed, parent r_lower_leg, child r_lower_leg_skin_21, origin xyz=0.0242704 0.0485378 -0.024277 rpy=2.29671149558e-05 -1.55545513881 -1.87411972316
- added joint r_lower_leg_skin_28_fixed_joint: type fixed, parent r_lower_leg, child r_lower_leg_skin_28, origin xyz=0.04087215 -0.04244 -0.032756 rpy=3.14158088865 -1.52252462169 -0.929681029763
- added joint r_lower_leg_skin_29_fixed_joint: type fixed, parent r_lower_leg, child r_lower_leg_skin_29, origin xyz=0.03846637 -0.043516 -0.05242 rpy=3.14158017044 -1.53429841563 -0.915436346631
- added joint r_lower_leg_skin_31_fixed_joint: type fixed, parent r_lower_leg, child r_lower_leg_skin_31, origin xyz=0.03914638 -0.042271 0.006327 rpy=-6.58381747139e-07 -1.4186494462 2.20853032986
- added joint r_lower_leg_skin_32_fixed_joint: type fixed, parent r_lower_leg, child r_lower_leg_skin_32, origin xyz=0.04598301 0.0325847 -0.080733 rpy=-3.14159014988 -1.52238289798 0.645940380887
- added joint r_lower_leg_skin_35_fixed_joint: type fixed, parent r_lower_leg, child r_lower_leg_skin_35, origin xyz=0.04774866 -0.031232 -0.080113 rpy=-3.14158668275 -1.51758467332 -0.541532486468
- added joint r_lower_leg_skin_36_fixed_joint: type fixed, parent r_lower_leg, child r_lower_leg_skin_36, origin xyz=0.05322409 -0.0156018 -0.088362 rpy=-3.14159034144 -1.51587265281 -0.20740733566
- added joint r_lower_leg_skin_37_fixed_joint: type fixed, parent r_lower_leg, child r_lower_leg_skin_37, origin xyz=0.0552572 0.0009644 -0.078318 rpy=-3.14158180452 -1.52318336898 0.00752450583063
- added joint r_lower_leg_skin_38_fixed_joint: type fixed, parent r_lower_leg, child r_lower_leg_skin_38, origin xyz=0.04880467 -0.031263 -0.060757 rpy=3.14158665199 -1.5157299554 -0.54215359959
- added joint r_lower_leg_skin_3_fixed_joint: type fixed, parent r_lower_leg, child r_lower_leg_skin_3, origin xyz=0.05157878 0.0304205 -0.002843 rpy=0 -1.42951054083 -2.30391484186
- added joint r_lower_leg_skin_41_fixed_joint: type fixed, parent r_lower_leg, child r_lower_leg_skin_41, origin xyz=0.0566009 -0.0159129 -0.049854 rpy=-3.14159198825 -1.40681343597 -0.248233089413
- added joint r_lower_leg_skin_42_fixed_joint: type fixed, parent r_lower_leg, child r_lower_leg_skin_42, origin xyz=0.0570106 0.0007962 -0.05908 rpy=3.14158970239 -1.43524750416 0.00687943651504
- added joint r_lower_leg_skin_43_fixed_joint: type fixed, parent r_lower_leg, child r_lower_leg_skin_43, origin xyz=0.04712542 0.0323653 -0.061362 rpy=-3.14159136621 -1.53843038237 0.624217523667
- added joint r_lower_leg_skin_46_fixed_joint: type fixed, parent r_lower_leg, child r_lower_leg_skin_46, origin xyz=0.0558156 0.0172164 -0.05018 rpy=-3.14158987809 -1.42759881603 0.325607710876
- added joint r_lower_leg_skin_47_fixed_joint: type fixed, parent r_lower_leg, child r_lower_leg_skin_47, origin xyz=0.05264163 0.0176389 -0.08886 rpy=3.14158963519 -1.51690559406 0.262640425058
- added joint r_lower_leg_skin_49_fixed_joint: type fixed, parent r_lower_leg, child r_lower_leg_skin_49, origin xyz=0.04113137 0.0324385 -0.138859 rpy=-3.14158934751 -1.48996135695 0.729763592113
- added joint r_lower_leg_skin_4_fixed_joint: type fixed, parent r_lower_leg, child r_lower_leg_skin_4, origin xyz=0.0583103 0.0167836 0.007272 rpy=-2.98636361519e-07 -1.25636748876 -2.75892380087
- added joint r_lower_leg_skin_50_fixed_joint: type fixed, parent r_lower_leg, child r_lower_leg_skin_50, origin xyz=0.043016947 0.0325273 -0.119469 rpy=3.14159069596 -1.49900732636 0.695784020081
- added joint r_lower_leg_skin_51_fixed_joint: type fixed, parent r_lower_leg, child r_lower_leg_skin_51, origin xyz=0.05141583 0.017759 -0.108206 rpy=-3.14158890179 -1.50628475717 0.272079935713
- added joint r_lower_leg_skin_52_fixed_joint: type fixed, parent r_lower_leg, child r_lower_leg_skin_52, origin xyz=0.05299832 0.0012664 -0.116895 rpy=-3.14159164042 -1.50318674421 0.0108717260994
- added joint r_lower_leg_skin_53_fixed_joint: type fixed, parent r_lower_leg, child r_lower_leg_skin_53, origin xyz=0.05207312 -0.0154339 -0.107654 rpy=3.14159063987 -1.50595307447 -0.211407322892
- added joint r_lower_leg_skin_54_fixed_joint: type fixed, parent r_lower_leg, child r_lower_leg_skin_54, origin xyz=0.04512708 -0.030749 -0.118787 rpy=3.14158825193 -1.49745145571 -0.575115374473
- added joint r_lower_leg_skin_55_fixed_joint: type fixed, parent r_lower_leg, child r_lower_leg_skin_55, origin xyz=0.043502663 -0.030489 -0.138143 rpy=3.14158906486 -1.48995787038 -0.597219943789
- added joint r_lower_leg_skin_56_fixed_joint: type fixed, parent r_lower_leg, child r_lower_leg_skin_56, origin xyz=0.04926839 -0.015121 -0.146218 rpy=-3.14158920404 -1.49124819828 -0.2234844764
- added joint r_lower_leg_skin_5_fixed_joint: type fixed, parent r_lower_leg, child r_lower_leg_skin_5, origin xyz=0.0636503 0.0003094 -0.001972 rpy=0 -1.38652215068 -3.14147169807
- added joint r_lower_leg_skin_60_fixed_joint: type fixed, parent r_lower_leg, child r_lower_leg_skin_60, origin xyz=0.04836967 0.018056 -0.146938 rpy=-3.14159173337 -1.48985968527 0.302951871954
- added joint r_lower_leg_skin_61_fixed_joint: type fixed, parent r_lower_leg, child r_lower_leg_skin_61, origin xyz=0.05161952 0.0014266 -0.136169 rpy=-3.14159100925 -1.49602097086 0.0132014275205
- added joint r_lower_leg_skin_6_fixed_joint: type fixed, parent r_lower_leg, child r_lower_leg_skin_6, origin xyz=0.05208552 0.0304434 -0.022149 rpy=-3.14158927953 -1.46785123411 0.837492889077
- added joint r_lower_leg_skin_9_fixed_joint: type fixed, parent r_lower_leg, child r_lower_leg_skin_9, origin xyz=0.0598214 0.0167973 -0.030962 rpy=-3.14159202356 -1.34224755325 0.379294477718
- added joint r_upper_leg_back_contact_fixed_joint: type fixed, parent r_upper_leg, child r_upper_leg_back_contact, origin xyz=-0.0511999 0 0.0146 rpy=0 1.57079632679 0
- added joint r_upper_leg_dh_frame_fixed_joint: type fixed, parent r_upper_leg, child r_upper_leg_dh_frame, origin xyz=0 0 -0.145825 rpy=1.57079632679 0 0
- joint l_ankle_pitch: axis 1.0 0.0 0.0 -> 2.22044604925e-16 1.0 0.0; limit lower=-0.523598775598 upper=0.523598775598 effort=50000 velocity=50000 -> lower=-0.610865238198 upper=0.610865238198 effort=50000 velocity=50000; origin xyz=0.0406034 -0.2005 0 rpy=0 0 0 -> xyz=0 0 -0.2005 rpy=0 0 0
- joint l_ankle_roll: axis 0.0 0.0 1.0 -> 1.0 0.0 2.22044604925e-16; limit lower=-0.349065850399 upper=0.349065850399 effort=50000 velocity=50000 -> lower=-0.436332312999 upper=0.436332312999 effort=50000 velocity=50000; origin xyz=-0.0270179 0 0.04808755 rpy=0 0 0 -> xyz=0 0 0 rpy=0 0 0
- joint l_foot_ft_sensor: origin xyz=0 -0.0603 -0.05158755 rpy=1.57079632679 -1.57079632679 0 -> xyz=-0.0035 0 -0.0605 rpy=3.14159265359 0 0
- joint l_hip_pitch: axis -1.0 0.0 0.0 -> -2.22044604925e-16 -1.0 0.0; limit lower=-0.523598775598 upper=1.4835298642 effort=50000 velocity=50000 -> lower=-0.785398163397 upper=2.33874119767 effort=50000 velocity=50000; origin xyz=0.0064515 -0.0223861 -0.119913 rpy=1.57079632679 0 -1.57079632679 -> xyz=0.0064515 -0.026 -0.119913 rpy=0 0 -3.14159265359
- joint l_hip_roll: axis 0.0 0.0 1.0 -> 1.0 0.0 2.22044604925e-16; limit lower=-0.261799 upper=1.48353 effort=50000 velocity=50000 -> lower=-0.349065850399 upper=2.09439510239 effort=50000 velocity=50000; origin xyz=0.0477139 0 -0.02554 rpy=0 0 0 -> xyz=0 0.0441 0 rpy=0 0 0
- joint l_hip_yaw: axis 0.0 1.0 0.0 -> 0.0 2.22044604925e-16 1.0; limit lower=-1.2217304764 upper=1.2217304764 effort=50000 velocity=50000 -> lower=-1.3962634016 upper=1.3962634016 effort=50000 velocity=50000; origin xyz=0 0 0.0146 rpy=-1.57079632679 0 -1.57079632679 -> xyz=0 0 0.0144 rpy=-3.14159265359 0 -1.57079632679
- joint l_knee: axis -1.0 0.0 0.0 -> -2.22044604925e-16 -1.0 -0.0; limit lower=-1.74532925199 upper=0.0 effort=50000 velocity=50000 -> lower=-2.16420827247 upper=0.0698131700798 effort=50000 velocity=50000; origin xyz=-0.0135855 -0.145625 0 rpy=0 0 0 -> xyz=0 0 -0.145825 rpy=0 0 0
- joint l_leg_ft_sensor: origin xyz=0 -0.0743 0.0246825 rpy=1.57079632679 -1.57079632679 0 -> xyz=-0.0008575 0 -0.0743 rpy=-3.14159265359 0 -1.57079632679
- joint r_ankle_pitch: axis 1.0 0.0 0.0 -> 2.22044604925e-16 1.0 0.0; limit lower=-0.523598775598 upper=0.523598775598 effort=50000 velocity=50000 -> lower=-0.610865238198 upper=0.610865238198 effort=50000 velocity=50000; origin xyz=-0.0188325 -0.2005 0 rpy=0 0 0 -> xyz=0 0 -0.2005 rpy=0 0 0
- joint r_ankle_roll: axis 0.0 0.0 -1.0 -> -1.0 -0.0 -2.22044604925e-16; limit lower=-0.349065850399 upper=0.349065850399 effort=50000 velocity=50000 -> lower=-0.436332312999 upper=0.436332312999 effort=50000 velocity=50000; origin xyz=0.0285 0 -0.0185 rpy=0 0 0 -> xyz=0 0 0 rpy=0 0 0
- joint r_foot_ft_sensor: origin xyz=0 -0.0603 0.015 rpy=1.57079632679 -1.57079632679 0 -> xyz=-0.0035 0 -0.0605 rpy=3.14159265359 0 0
- joint r_hip_pitch: axis -1.0 0.0 0.0 -> -2.22044604925e-16 -1.0 -0.0; limit lower=-0.523598775598 upper=1.4835298642 effort=50000 velocity=50000 -> lower=-0.785398163397 upper=2.33874119767 effort=50000 velocity=50000; origin xyz=0.0064515 0.0233655 -0.119913 rpy=1.57079632679 0 -1.57079632679 -> xyz=0.0064515 0.026 -0.119913 rpy=0 0 -3.14159265359
- joint r_hip_roll: axis 0.0 0.0 -1.0 -> -1.0 0.0 -2.22044604925e-16; limit lower=-0.261799 upper=1.48353 effort=50000 velocity=50000 -> lower=-0.349065850399 upper=2.09439510239 effort=50000 velocity=50000; origin xyz=-0.0467345 0 -0.0263447 rpy=0 0 0 -> xyz=0 -0.0441 0 rpy=0 0 0
- joint r_hip_yaw: axis 0.0 -1.0 0.0 -> 0.0 -2.22044604925e-16 -1.0; limit lower=-1.2217304764 upper=1.2217304764 effort=50000 velocity=50000 -> lower=-1.3962634016 upper=1.3962634016 effort=50000 velocity=50000; origin xyz=0 0 0.0146 rpy=-1.57079632679 0 -1.57079632679 -> xyz=0 0 0.0144 rpy=-3.14159265359 0 0
- joint r_knee: axis -1.0 0.0 0.0 -> -2.22044604925e-16 -1.0 0.0; limit lower=-1.74532925199 upper=0.0 effort=50000 velocity=50000 -> lower=-2.16420827247 upper=0.0698131700798 effort=50000 velocity=50000; origin xyz=-0.0096675 -0.145625 0 rpy=0 0 0 -> xyz=0 0 -0.145825 rpy=0 0 0
- joint r_leg_ft_sensor: origin xyz=0 -0.0743 0.0254872 rpy=1.57079632679 -1.57079632679 0 -> xyz=-0.0008575 0 -0.0743 rpy=3.14159265359 0 0

Commit message: updated robot model

File: resources/models/iCubGenova04.urdf (robot description, URDF)
Before this commit: robot iCub, 139 links, 138 joints
Joints:
- joint l_ankle_pitch: limit lower=-0.610865238198 upper=0.610865238198 effort=50000 velocity=50000 -> lower=-0.610865238198 upper=0.610865238198 effort=37.0 velocity=7.64
- joint l_ankle_roll: limit lower=-0.436332312999 upper=0.436332312999 effort=50000 velocity=50000 -> lower=-0.436332312999 upper=0.436332312999 effort=37.0 velocity=7.64
- joint l_hip_pitch: limit lower=-0.785398163397 upper=2.33874119767 effort=50000 velocity=50000 -> lower=-0.785398163397 upper=2.33874119767 effort=55.5 velocity=5.1
- joint l_hip_roll: limit lower=-0.349065850399 upper=2.09439510239 effort=50000 velocity=50000 -> lower=-0.349065850399 upper=2.09439510239 effort=37.0 velocity=7.64
- joint l_hip_yaw: limit lower=-1.3962634016 upper=1.3962634016 effort=50000 velocity=50000 -> lower=-1.3962634016 upper=1.3962634016 effort=37.0 velocity=7.64
- joint l_knee: limit lower=-2.16420827247 upper=0.0698131700798 effort=50000 velocity=50000 -> lower=-2.16420827247 upper=0.0698131700798 effort=37.0 velocity=7.64
- joint r_ankle_pitch: limit lower=-0.610865238198 upper=0.610865238198 effort=50000 velocity=50000 -> lower=-0.610865238198 upper=0.610865238198 effort=37.0 velocity=7.64
- joint r_ankle_roll: limit lower=-0.436332312999 upper=0.436332312999 effort=50000 velocity=50000 -> lower=-0.436332312999 upper=0.436332312999 effort=37.0 velocity=7.64
- joint r_hip_pitch: limit lower=-0.785398163397 upper=2.33874119767 effort=50000 velocity=50000 -> lower=-0.785398163397 upper=2.33874119767 effort=55.5 velocity=5.1
- joint r_hip_roll: limit lower=-0.349065850399 upper=2.09439510239 effort=50000 velocity=50000 -> lower=-0.349065850399 upper=2.09439510239 effort=37.0 velocity=7.64
- joint r_hip_yaw: limit lower=-1.3962634016 upper=1.3962634016 effort=50000 velocity=50000 -> lower=-1.3962634016 upper=1.3962634016 effort=37.0 velocity=7.64
- joint r_knee: limit lower=-2.16420827247 upper=0.0698131700798 effort=50000 velocity=50000 -> lower=-2.16420827247 upper=0.0698131700798 effort=37.0 velocity=7.64
