Commit message: Fix model orientation and remove custom rotations.

File: resources/models/iCubGenova04.urdf (robot description, URDF)
Before this commit: robot iCub, 139 links, 138 joints
Joints:
- joint base_fixed_joint: origin xyz=0 0 0 rpy=0 -0 0 -> xyz=0 0 0 rpy=0 -0 3.14

Commit message: Add more decimal digits to pi to avoid approximation errors.

File: resources/models/iCubGenova04.urdf (robot description, URDF)
Before this commit: robot iCub, 139 links, 138 joints
Joints:
- joint base_fixed_joint: origin xyz=0 0 0 rpy=0 -0 3.14 -> xyz=0 0 0 rpy=0 -0 3.14159265358979323846
